File: 5V-3.3V pawah.kicad_pcb (KiCad board)
At the start: 2 copper layers, 61.7 x 53.8 mm, 17 parts, among them J1 Barrel_Jack_Switch, J2 Conn_01x02_Male, J3 Conn_01x02_Male, U1 LM7805_TO220, U3 LM317_TO-220

Commit message: Update PCB
Parts:
- added HS1: Heatsink, TO_SOT_Packages_THT:Heatsink_TO220, F.Cu at (143.0, 75.2)
- moved J3 2.86 mm to (120.4, 104.9), turned to 90 degrees
- moved R10 1.52 mm to (126.0, 95.5)
Routing:
- net GND: track 204.9 -> 217.0 mm
- net +5V: track 126.2 -> 128.2 mm
- net Net-(D3-Pad2): track 5.84 -> 7.37 mm
- net +12V: track 34.0 -> 35.1 mm
Other:
- board text added: "- + 5V"
- board text added: "3.3V - +"
