File: 5V-3.3V pawah.sch (KiCad schematic (older format))
At the start: 17 parts, among them J1 Barrel_Jack_Switch, J2 Conn_01x02_Male, J3 Conn_01x02_Male, U1 LM7805_TO220, U3 LM317_TO-220

Commit message: Update PCB
Parts:
- added HS1: Heatsink, TO_SOT_Packages_THT:Heatsink_TO220, symbol Mechanical:Heatsink
Changed lines of the file:
@@
 	3200 2450 3200 2550
 Connection ~ 3200 2550
+$Comp
+L Mechanical:Heatsink HS1
+U 1 1 62AE3852
+P 5400 2550
+F 0 "HS1" H 5542 2671 50  0000 L CNN
+F 1 "Heatsink" H 5542 2580 50  0000 L CNN
+F 2 "TO_SOT_Packages_THT:Heatsink_TO220" H 5412 2550 50  0001 C CNN
+F 3 "~" H 5412 2550 50  0001 C CNN
+	1    5400 2550
+	1    0    0    -1
+$EndComp
 $EndSCHEMATC
